Commit message: change to ddbot_pkg and add ros2 control gazebo

File: ddbot_pkg/urdf/ddbot_description.xacro (robot description, xacro)
@@ -83,5 +83,5 @@
         <origin xyz="0 0 0" rpy="${pi/2} 0 0"/>
         <geometry>
-          <cylinder radius="${wheel_radius}" length="${wheel_width}"/>
+          <sphere radius="${wheel_radius}"/>
         </geometry>
       </collision>

File: urdf_pkg/urdf/diff_drive_robot_urdf.xacro (robot description, xacro)
@@ -2,4 +2,4 @@
 <robot name="diff_drive_robot" xmlns:xacro="http://www.ros.org/wiki/xacro">
   <xacro:include filename="diff_drive_robot_description.xacro" />
-  <xacro:include filename="diff_drive_robot_gazebo.xacro" />
+  <xacro:include filename="diff_drive_robot_control.xacro" />
 </robot>

Commit message: add sim_camera and sim_lidar

File: ddbot_pkg/urdf/ddbot_description.xacro (robot description, xacro)
@@ -125,48 +125,3 @@
         <mu2 value="0.001"/>
   </gazebo>
-  <!-- lidar -->
-  <link name="lidar_link">
-    <visual>
-      <origin xyz="0 0 0" rpy="0 0 0"/>
-      <geometry>
-        <cylinder radius="0.0737" length="0.0425"/>
-      </geometry>
-      <material name="blue"/>
-    </visual>
-    <collision>
-      <origin xyz="0 0 0" rpy="0 0 0"/>
-      <geometry>
-        <cylinder radius="0.0737" length="0.0425"/>
-      </geometry>
-    </collision>
-    <xacro:cylinder_inertia m="0.5" r="0.0737" h="0.0425"/>
-  </link>
-  <joint name="lidar_joint" type="fixed">
-    <parent link="body_link"/>
-    <child link="lidar_link"/>
-    <origin xyz="0 0 0.03685" rpy="0 0 0"/>
-  </joint>
-  <gazebo reference="lidar_link"><material>Gazebo/Blue</material></gazebo>
-  <!-- CAMERA LINK -->
-  <link name="camera_link">
-    <visual>
-      <geometry>
-        <box size="0.025 0.023 0.009"/>
-      </geometry>
-      <origin xyz="0 0 0" rpy="0 1.5708 0"/>
-      <material name="blue"/>
-    </visual>
-    <collision>
-      <geometry>
-        <box size="0.025 0.023 0.009"/>
-      </geometry>
-    </collision>
-    <xacro:box_inertia m="0.1" w="0.025" d="0.023" h="0.009"/>
-  </link>
-  <joint name="camera_joint" type="fixed">
-      <parent link="body_link"/>
-      <child link="camera_link"/>
-      <origin xyz="0.12 0 0"/>
-  </joint>
-  <gazebo reference="camera_link"><material>Gazebo/Blue</material></gazebo>
 </robot>

File: ddbot_pkg/urdf/ddbot_urdf.xacro (robot description, xacro)
@@ -3,4 +3,6 @@
   <xacro:arg name="use_ros2_control" default="true"/>
   <xacro:include filename="ddbot_description.xacro" />
+  <xacro:include filename="ddbot_lidar.xacro" />
+  <xacro:include filename="ddbot_camera.xacro" />
   <xacro:if value="$(arg use_ros2_control)">
       <xacro:include filename="ddbot_control.xacro" />

Commit message: change robot size and move wheel to center

File: ddbot_pkg/urdf/ddbot_description.xacro (robot description, xacro)
@@ -9,9 +9,8 @@
   <xacro:property name="base_length" value="0.24"/>
   <xacro:property name="base_height" value="0.05"/>
-  <xacro:property name="base_zoff" value="0.105"/>
   <xacro:property name="wheel_radius" value="0.0435"/>
   <xacro:property name="wheel_width" value="0.04"/>
-  <xacro:property name="wheel_ygap" value="0.025"/>
-  <xacro:property name="wheel_zoff" value="0.0615"/>
+  <xacro:property name="wheel_ygap" value="0.03"/>
+  <xacro:property name="wheel_zoff" value="0.034"/>
   <xacro:property name="wheel_xoff" value="0.07"/>
   <xacro:property name="caster_xoff" value="0.1"/>
@@ -67,5 +66,5 @@
     <parent link="base_link"/>
     <child link="body_link"/>
-    <origin xyz="0.0 0.0 ${base_zoff}" rpy="0 0 0"/>
+    <origin xyz="0.0 0.0 ${wheel_zoff+wheel_radius}" rpy="0 0 0"/>
   </joint>
   <gazebo reference="base_link"><material>Gazebo/White</material></gazebo>
@@ -91,5 +90,5 @@
       <parent link="body_link"/>
       <child link="${prefix}_link"/>
-      <origin xyz="${x_reflect*wheel_xoff} ${y_reflect*(base_width/2+wheel_ygap)} ${-wheel_zoff}" rpy="0 0 0"/>
+      <origin xyz="0 ${y_reflect*(base_width/2+wheel_ygap)} ${-wheel_zoff}" rpy="0 0 0"/>
       <axis xyz="0 1 0"/>
     </joint>
@@ -113,5 +112,5 @@
       </geometry>
     </collision>
-    <xacro:sphere_inertia m="0.5" r="${wheel_radius}"/>
+    <xacro:sphere_inertia m="0.01" r="${wheel_radius}"/>
   </link>
   <joint name="caster_joint" type="fixed">

File: ddbot_pkg/urdf/ddbot_gazebo.xacro (robot description, xacro)
@@ -7,5 +7,5 @@
         <right_joint>right_wheel_joint</right_joint>
         <!-- kinematics -->
-        <wheel_separation>0.35</wheel_separation>
+        <wheel_separation>0.36</wheel_separation>
         <wheel_diameter>0.087</wheel_diameter>
         <!-- Limits -->
