Commit message: fix ros2_control odometry and color

File: ddbot_pkg/urdf/ddbot_camera.xacro (robot description, xacro)
@@ -44,4 +44,4 @@
       </plugin>
     </sensor>
-    </gazebo>
+  </gazebo>
 </robot>

File: ddbot_pkg/urdf/ddbot_description.xacro (robot description, xacro)
@@ -90,5 +90,5 @@
       <parent link="body_link"/>
       <child link="${prefix}_link"/>
-      <origin xyz="0 ${y_reflect*(base_width/2+wheel_ygap)} ${-wheel_zoff}" rpy="0 0 0"/>
+      <origin xyz="${x_reflect*wheel_xoff} ${y_reflect*(base_width/2+wheel_ygap)} ${-wheel_zoff}" rpy="0 0 0"/>
       <axis xyz="0 1 0"/>
     </joint>

File: ddbot_pkg/urdf/ddbot_lidar.xacro (robot description, xacro)
@@ -24,4 +24,5 @@
   </joint>
   <gazebo reference="lidar_link">
+    <material>Gazebo/Blue</material>
     <sensor name="lidar" type="ray">
       <visualize>false</visualize>
